Commit message: feat: add HexPercept1

File: hexapod_elevation_mapping/model/modules/HexPercept1/HexPercept1.xacro (robot description, xacro)
@@ -1,5 +1,5 @@
 <?xml version="1.0"?>
 <robot xmlns:xacro="http://www.ros.org/wiki/xacro">
-    <xacro:macro name="SensorModuleVer1" params="parent_link *origin">
+    <xacro:macro name="HexPercept1" params="parent_link *origin">
         <!-- Const -->
         <xacro:arg name="gpu" default="false"/>
@@ -25,5 +25,5 @@
                 <origin xyz="0 0 0" rpy="0 0 0" />
                 <geometry>
-                    <mesh filename="package://hexapod_elevation_mapping/model/sensor_assembly/sensor_module_ver1/sensorSupport.STL"/>
+                    <mesh filename="package://hexapod_elevation_mapping/model/modules/HexPercept1/sensorSupport.STL"/>
                 </geometry>
                 <material name="">
@@ -34,5 +34,5 @@
                 <origin xyz="0 0 0" rpy="0 0 0" />
                 <geometry>
-                    <mesh filename="package://hexapod_elevation_mapping/model/sensor_assembly/sensor_module_ver1/sensorSupport.STL"/>
+                    <mesh filename="package://hexapod_elevation_mapping/model/modules/HexPercept1/sensorSupport.STL"/>
                 </geometry>
             </collision>

Commit message: feat: BPearl lidar gazebo demo

File: hexapod_elevation_mapping/model/modules/HexPercept1/HexPercept1.xacro (robot description, xacro)
@@ -1,5 +1,5 @@
 <?xml version="1.0"?>
 <robot xmlns:xacro="http://www.ros.org/wiki/xacro">
-    <xacro:macro name="HexPercept1" params="parent_link *origin">
+    <xacro:macro name="HexPercept1" params="parent_link *origin lidar_frame_name:=velodyneLidar camera_frame_name:=camera">
         <!-- Const -->
         <xacro:arg name="gpu" default="false"/>
@@ -39,9 +39,9 @@
         </link>
         <xacro:include filename="$(find hexapod_elevation_mapping)/model/sensors/VLP-16/xacro/VLP-16.urdf.xacro"/>
-        <xacro:VLP-16 parent="sensorSupport" name="velodyneLidar" topic="/velodyne_points" organize_cloud="${organize_cloud}" hz="10" samples="220" gpu="${gpu}">
+        <xacro:VLP-16 parent="sensorSupport" name="${lidar_frame_name}" topic="/velodyne_points" organize_cloud="${organize_cloud}" hz="10" samples="220" gpu="${gpu}">
             <origin xyz="0 -0.13 0" rpy="1.5708 1.5708 -0.25" />
         </xacro:VLP-16>
         <xacro:include filename="$(find realsense_ros_gazebo)/xacro/tracker.xacro"/>
-        <xacro:realsense_T265 sensor_name="T265_camera" parent_link="sensorSupport" rate="30.0">
+        <xacro:realsense_T265 sensor_name="${camera_frame_name}" parent_link="sensorSupport" rate="30.0">
             <origin rpy="-1.5708 0 ${3.14159 - 0.395}" xyz="-0.12 -0.04 0"/>
         </xacro:realsense_T265>

File: hexapod_elevation_mapping/model/modules/HexPercept1/example.xacro (robot description, xacro)
@@ -1,7 +1,9 @@
 <?xml version="1.0"?>
 <robot name="HexPercept1_example" xmlns:xacro="http://www.ros.org/wiki/xacro">
+    <xacro:property name="lidar_frame_name" value="velodyneLidar"/>
+    <xacro:property name="camera_frame_name" value="camera"/>
     <link name="base_link"/>
     <xacro:include filename="$(find hexapod_elevation_mapping)/model/modules/HexPercept1/HexPercept1.xacro"/>
-    <xacro:HexPercept1 parent_link="base_link">
+    <xacro:HexPercept1 parent_link="base_link" lidar_frame_name="${lidar_frame_name}" camera_frame_name="${camera_frame_name}">
         <origin rpy="-1.5708 0 3.1415" xyz="0 0 0"/>
     </xacro:HexPercept1>

File: hexapod_elevation_mapping/model/modules/HexPercept2/HexPercept2.xacro (robot description, xacro)
@@ -1,5 +1,5 @@
 <?xml version="1.0"?>
 <robot xmlns:xacro="http://www.ros.org/wiki/xacro">
-    <xacro:macro name="HexPercept2" params="parent_link *origin">
+    <xacro:macro name="HexPercept2" params="parent_link *origin lidar_frame_name:=BPearl_Lidar camera_frame_name:=camera">
         <!-- Const -->
         <xacro:arg name="gpu" default="false"/>
@@ -41,9 +41,9 @@
         </link>
         <xacro:include filename="$(find hexapod_elevation_mapping)/model/sensors/RS-BPearl/xacro/RS-BPearl.xacro"/>
-        <xacro:RS-BPearl parent="sensorSupport" name="RS-BPearlLidar" topic="/bpearl_points2" organize_cloud="${organize_cloud}" hz="15" samples="1000" gpu="${gpu}">
-            <origin xyz="0 0 0" rpy="0 0 0" />
+        <xacro:RS-BPearl parent="sensorSupport" name="${lidar_frame_name}" topic="/bpearl_points" organize_cloud="${organize_cloud}" hz="15" samples="1000" gpu="${gpu}">
+            <origin xyz="0 0 0" rpy="0 1.5708 0" />
         </xacro:RS-BPearl>
         <xacro:include filename="$(find realsense_ros_gazebo)/xacro/tracker.xacro"/>
-        <xacro:realsense_T265 sensor_name="T265_camera" parent_link="sensorSupport" rate="30.0">
+        <xacro:realsense_T265 sensor_name="${camera_frame_name}" parent_link="sensorSupport" rate="30.0">
             <origin rpy="0 0 0" xyz="0.0026 0 0.06854"/>
         </xacro:realsense_T265>

File: hexapod_elevation_mapping/model/modules/HexPercept2/example.xacro (robot description, xacro)
@@ -1,7 +1,9 @@
 <?xml version="1.0"?>
 <robot name="HexPercept2_example" xmlns:xacro="http://www.ros.org/wiki/xacro">
+    <xacro:property name="lidar_frame_name" value="BPearl_Lidar"/>
+    <xacro:property name="camera_frame_name" value="camera"/>
     <link name="base_link"/>
     <xacro:include filename="$(find hexapod_elevation_mapping)/model/modules/HexPercept2/HexPercept2.xacro"/>
-    <xacro:HexPercept2 parent_link="base_link">
+    <xacro:HexPercept2 parent_link="base_link" lidar_frame_name="${lidar_frame_name}" camera_frame_name="${camera_frame_name}">
         <origin rpy="0 0 0" xyz="0 0 0"/>
     </xacro:HexPercept2>

File: hexapod_elevation_mapping/model/sensors/RS-BPearl/xacro/RS-BPearl.xacro (robot description, xacro)
@@ -11,5 +11,5 @@
       <inertial>
         <mass value="0.83"/>
-        <origin xyz="0 0 0.03585"/>
+        <origin rpy="0 0 0" xyz="0 0 0.055"/>
         <inertia ixx="${(0.83 * (3.0*0.0516*0.0516 + 0.0717*0.0717)) / 12.0}" ixy="0" ixz="0"
           iyy="${(0.83 * (3.0*0.0516*0.0516 + 0.0717*0.0717)) / 12.0}" iyz="0"
@@ -20,14 +20,15 @@
           <mesh filename="package://hexapod_elevation_mapping/model/sensors/RS-BPearl/meshes/BPearl.STL" />
         </geometry>
+        <origin rpy="0 -1.5708 0" xyz="0 0 0"/>
       </visual>
       <collision>
-        <origin rpy="0 0 0" xyz="0 0 0.03585"/>
+        <origin rpy="0 0 0" xyz="0 0 0.055"/>
         <geometry>
-          <cylinder radius="0.0516" length="0.0717"/>
+          <cylinder radius="0.0500" length="0.11"/>
         </geometry>
       </collision>
     </link>
     <joint name="${name}_base_scan_joint" type="fixed" >
-      <origin xyz="0 0 0.0377" rpy="0 0 0" />
+      <origin xyz="0 0 0.07" rpy="0 0 0" />
       <parent link="${name}_base_link" />
       <child link="${name}"/>

Commit message: doc: update

File: hexapod_elevation_mapping/model/modules/HexPercept1/HexPercept1.xacro (robot description, xacro)
@@ -20,5 +20,5 @@
                 <mass value="30.0"/>
                 <!-- FIXME: need to update ixx,iyy and izz -->
-                <inertia ixx="0.1" ixy="0.0" ixz="0.0" iyy="0.1" iyz="0.0" izz="0.1}"/>
+                <inertia ixx="0.1" ixy="0.0" ixz="0.0" iyy="0.1" iyz="0.0" izz="0.1"/>
             </inertial>
             <visual>
