Commit message: fix: izz invalid

File: hexapod_elevation_mapping/model/modules/HexPercept2/HexPercept2.xacro (robot description, xacro)
@@ -20,5 +20,5 @@
                 <mass value="1.0"/>
                 <!-- FIXME: need to update ixx,iyy and izz -->
-                <inertia ixx="0.1" ixy="0.0" ixz="0.0" iyy="0.1" iyz="0.0" izz="0.1}"/>
+                <inertia ixx="0.1" ixy="0.0" ixz="0.0" iyy="0.1" iyz="0.0" izz="0.1"/>
             </inertial>
             <visual>

File: hexapod_elevation_mapping/model/modules/HexPercept3/HexPercept3.xacro (robot description, xacro)
@@ -20,5 +20,5 @@
                 <mass value="1.0"/>
                 <!-- FIXME: need to update ixx,iyy and izz -->
-                <inertia ixx="0.1" ixy="0.0" ixz="0.0" iyy="0.1" iyz="0.0" izz="0.1}"/>
+                <inertia ixx="0.1" ixy="0.0" ixz="0.0" iyy="0.1" iyz="0.0" izz="0.1"/>
             </inertial>
             <visual>
