Commit message: feat: add HexPercept3 demo

File: hexapod_elevation_mapping/model/modules/HexPercept3/HexPercept3.xacro (robot description, xacro)
@@ -1,5 +1,5 @@
 <?xml version="1.0"?>
 <robot xmlns:xacro="http://www.ros.org/wiki/xacro">
-    <xacro:macro name="HexPercept2" params="parent_link *origin lidar_frame_name:=BPearl_Lidar camera_frame_name:=camera">
+    <xacro:macro name="HexPercept3" params="parent_link *origin lidar_frame_name:=BPearl_Lidar camera_frame_name:=camera">
         <!-- Const -->
         <xacro:arg name="gpu" default="false"/>
@@ -25,5 +25,5 @@
                 <origin xyz="0 0 0" rpy="0 0 0" />
                 <geometry>
-                    <mesh filename="package://hexapod_elevation_mapping/model/modules/HexPercept2/Support.STL"/>
+                    <mesh filename="package://hexapod_elevation_mapping/model/modules/HexPercept3/Support.STL"/>
                     <!-- Scale down 1000 times -->
                     <scale xyz="0.001 0.001 0.001"/>
@@ -36,5 +36,5 @@
                 <origin xyz="0 0 0" rpy="0 0 0" />
                 <geometry>
-                    <mesh filename="package://hexapod_elevation_mapping/model/modules/HexPercept2/Support.STL"/>
+                    <mesh filename="package://hexapod_elevation_mapping/model/modules/HexPercept3/Support.STL"/>
                 </geometry>
             </collision>
@@ -42,9 +42,9 @@
         <xacro:include filename="$(find hexapod_elevation_mapping)/model/sensors/RS-BPearl/xacro/RS-BPearl.xacro"/>
         <xacro:RS-BPearl parent="sensorSupport" name="${lidar_frame_name}" topic="/bpearl_points" organize_cloud="${organize_cloud}" hz="15" samples="1000" gpu="${gpu}">
-            <origin xyz="0 0 0" rpy="0 1.5708 0" />
+            <origin xyz="-0.045 0 0.15" rpy="0 1.5708 0" />
         </xacro:RS-BPearl>
         <xacro:include filename="$(find realsense_ros_gazebo)/xacro/tracker.xacro"/>
         <xacro:realsense_T265 sensor_name="${camera_frame_name}" parent_link="sensorSupport" rate="30.0">
-            <origin rpy="0 0 0" xyz="0.0026 0 0.06854"/>
+            <origin rpy="0 0 0" xyz="0.0125 0 0.014"/>
         </xacro:realsense_T265>
     </xacro:macro>

Commit message: chore: update param

File: hexapod_elevation_mapping/model/modules/HexPercept3/HexPercept3.xacro (robot description, xacro)
@@ -20,5 +20,5 @@
                 <mass value="1.0"/>
                 <!-- FIXME: need to update ixx,iyy and izz -->
-                <inertia ixx="0.1" ixy="0.0" ixz="0.0" iyy="0.1" iyz="0.0" izz="0.1"/>
+                <inertia ixx="0.01" ixy="0.0" ixz="0.0" iyy="0.01" iyz="0.0" izz="0.01"/>
             </inertial>
             <visual>
