Commit message: gai

File: hexapod_elevation_mapping/model/modules/MetaCam/MetaCam.xacro (robot description, xacro)
@@ -25,5 +25,5 @@
                 <origin xyz="0 0 0" rpy="0 0 0" />
                 <geometry>
-                    <mesh filename="package://hexapod_elevation_mapping/model/modules/HexPercept3_vins/Support.STL"/>
+                    <mesh filename="package://hexapod_elevation_mapping/model/modules/MetaCam/Support.STL"/>
                 </geometry>
                 <material name="">
@@ -34,5 +34,5 @@
                 <origin xyz="0 0 0" rpy="0 0 0" />
                 <geometry>
-                    <mesh filename="package://hexapod_elevation_mapping/model/modules/HexPercept3_vins/Support.STL"/>
+                    <mesh filename="package://hexapod_elevation_mapping/model/modules/MetaCam/Support.STL"/>
                 </geometry>
             </collision>
